File: PCBs/Recovery Board.kicad_pcb (KiCad board)
At the start: 2 copper layers, 73.7 x 50.8 mm, 21 parts, among them U1 R-78E3.3-0.5, X1 XBee-S2C

Commit message: Fixed grounds and missing terminal
Routing:
- net GoPro_Power: track 10.4 -> 21.5 mm
- net GND: track 0.00 -> 10.3 mm, vias 0 -> 5
- net Net-(A1-Pad16): track 35.1 -> 26.5 mm
- net Net-(R1-Pad1): track 0.00 -> 3.47 mm
Changed lines of the file:
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@@
   (general
     (links 31)
-    (no_connects 7)
+    (no_connects 0)
     (area 93.904999 98.984999 167.715001 149.935001)
     (thickness 1.6)
-    (drawings 17)
-    (tracks 54)
+    (drawings 22)
+    (tracks 67)
     (zones 0)
     (modules 21)
@@
       (xy -0.001755 -2.811832) (xy 0.000023 -2.81432) (xy 0.002958 -2.809977)) (layer F.SilkS) (width 0.01))
   )
+  (dimension 43.18 (width 0.3) (layer F.SilkS)
+    (gr_text "43.180 mm" (at 176.356 124.46 90) (layer F.SilkS)
+      (effects (font (size 1.5 1.5) (thickness 0.3)))
+    )
+    (feature1 (pts (xy 163.83 102.87) (xy 177.706 102.87)))
+    (feature2 (pts (xy 163.83 146.05) (xy 177.706 146.05)))
+    (crossbar (pts (xy 175.006 146.05) (xy 175.006 102.87)))
+    (arrow1a (pts (xy 175.006 102.87) (xy 175.592421 103.996504)))
+    (arrow1b (pts (xy 175.006 102.87) (xy 174.419579 103.996504)))
+    (arrow2a (pts (xy 175.006 146.05) (xy 175.592421 144.923496)))
+    (arrow2b (pts (xy 175.006 146.05) (xy 174.419579 144.923496)))
+  )
+  (dimension 3.81 (width 0.3) (layer F.SilkS)
+    (gr_text "3.810 mm" (at 165.735 83.486) (layer F.SilkS)
+      (effects (font (size 1.5 1.5) (thickness 0.3)))
+    )
+    (feature1 (pts (xy 167.64 102.87) (xy 167.64 82.136)))
+    (feature2 (pts (xy 163.83 102.87) (xy 163.83 82.136)))
+    (crossbar (pts (xy 163.83 84.836) (xy 167.64 84.836)))
+    (arrow1a (pts (xy 167.64 84.836) (xy 166.513496 85.422421)))
+    (arrow1b (pts (xy 167.64 84.836) (xy 166.513496 84.249579)))
+    (arrow2a (pts (xy 163.83 84.836) (xy 164.956504 85.422421)))
+    (arrow2b (pts (xy 163.83 84.836) (xy 164.956504 84.249579)))
+  )
+  (dimension 3.81 (width 0.3) (layer F.SilkS)
+    (gr_text "3.810 mm" (at 198.708 100.965 90) (layer F.SilkS)
+      (effects (font (size 1.5 1.5) (thickness 0.3)))
+    )
+    (feature1 (pts (xy 163.83 99.06) (xy 200.058 99.06)))
+    (feature2 (pts (xy 163.83 102.87) (xy 200.058 102.87)))
+    (crossbar (pts (xy 197.358 102.87) (xy 197.358 99.06)))
+    (arrow1a (pts (xy 197.358 99.06) (xy 197.944421 100.186504)))
+    (arrow1b (pts (xy 197.358 99.06) (xy 196.771579 100.186504)))
+    (arrow2a (pts (xy 197.358 102.87) (xy 197.944421 101.743496)))
+    (arrow2b (pts (xy 197.358 102.87) (xy 196.771579 101.743496)))
+  )
+  (dimension 50.8 (width 0.3) (layer F.SilkS)
+    (gr_text "50.800 mm" (at 190.326 124.46 270) (layer F.SilkS)
+      (effects (font (size 1.5 1.5) (thickness 0.3)))
+    )
+    (feature1 (pts (xy 167.64 149.86) (xy 191.676 149.86)))
+    (feature2 (pts (xy 167.64 99.06) (xy 191.676 99.06)))
+    (crossbar (pts (xy 188.976 99.06) (xy 188.976 149.86)))
+    (arrow1a (pts (xy 188.976 149.86) (xy 188.389579 148.733496)))
+    (arrow1b (pts (xy 188.976 149.86) (xy 189.562421 148.733496)))
+    (arrow2a (pts (xy 188.976 99.06) (xy 188.389579 100.186504)))
+    (arrow2b (pts (xy 188.976 99.06) (xy 189.562421 100.186504)))
+  )
+  (dimension 73.66 (width 0.3) (layer F.SilkS)
+    (gr_text "73.660 mm" (at 130.81 88.058001) (layer F.SilkS)
+      (effects (font (size 1.5 1.5) (thickness 0.3)))
+    )
+    (feature1 (pts (xy 93.98 99.06) (xy 93.98 86.708001)))
+    (feature2 (pts (xy 167.64 99.06) (xy 167.64 86.708001)))
+    (crossbar (pts (xy 167.64 89.408001) (xy 93.98 89.408001)))
+    (arrow1a (pts (xy 93.98 89.408001) (xy 95.106504 88.82158)))
+    (arrow1b (pts (xy 93.98 89.408001) (xy 95.106504 89.994422)))
+    (arrow2a (pts (xy 167.64 89.408001) (xy 166.513496 88.82158)))
+    (arrow2b (pts (xy 167.64 89.408001) (xy 166.513496 89.994422)))
+  )
   (gr_text "Adam Paul" (at 146.812 102.616) (layer F.SilkS)
     (effects (font (size 1 1) (thickness 0.15)) (justify left))
@@
   (segment (start 128.27 116.84) (end 121.92 116.84) (width 0.25) (layer F.Cu) (net 2))
   (segment (start 128.27 116.84) (end 128.27 116.84) (width 0.25) (layer F.Cu) (net 2))
+  (segment (start 125.71 114.3) (end 128.016 114.3) (width 0.25) (layer F.Cu) (net 3) (status 400000))
+  (via (at 128.016 114.3) (size 0.6) (drill 0.4) (layers F.Cu B.Cu) (net 3))
+  (segment (start 133.33 114.3) (end 135.636 114.3) (width 0.25) (layer F.Cu) (net 3) (status 400000))
+  (via (at 135.636 114.3) (size 0.6) (drill 0.4) (layers F.Cu B.Cu) (net 3))
+  (segment (start 123.11 119.38) (end 123.11 120.316) (width 0.25) (layer F.Cu) (net 3) (status 400000))
+  (via (at 123.952 121.158) (size 0.6) (drill 0.4) (layers F.Cu B.Cu) (net 3))
+  (segment (start 123.11 120.316) (end 123.952 121.158) (width 0.25) (layer F.Cu) (net 3))
+  (segment (start 127 129.28) (end 127 127.508) (width 0.25) (layer F.Cu) (net 3))
+  (via (at 127 127.508) (size 0.6) (drill 0.4) (layers F.Cu B.Cu) (net 3))
+  (segment (start 133.35 129.28) (end 133.35 127.508) (width 0.25) (layer F.Cu) (net 3))
+  (via (at 133.35 127.508) (size 0.6) (drill 0.4) (layers F.Cu B.Cu) (net 3))
   (segment (start 139.8778 113.57356) (end 136.94156 113.57356) (width 0.25) (layer B.Cu) (net 4))
   (segment (start 106.172 102.108) (end 104.14 104.14) (width 0.25) (layer B.Cu) (net 4))
@@
   (segment (start 123.19 123.19) (end 121.92 123.19) (width 0.25) (layer F.Cu) (net 29))
   (segment (start 130.81 123.19) (end 124.46 123.11) (width 0.25) (layer F.Cu) (net 29) (status 10))
-  (segment (start 130.81 125.73) (end 130.81 123.19) (width 0.25) (layer F.Cu) (net 29) (status 30))
-  (segment (start 130.81 123.19) (end 130.81 129.28) (width 0.25) (layer F.Cu) (net 29) (status 10))
   (segment (start 130.81 109.22) (end 137.52576 109.22) (width 0.25) (layer F.Cu) (net 30))
   (segment (start 137.52576 109.22) (end 139.8778 111.57204) (width 0.25) (layer F.Cu) (net 30))
@@
   (segment (start 130.81 111.76) (end 130.81 114.28) (width 0.25) (layer F.Cu) (net 30) (status 20))
   (segment (start 130.81 114.28) (end 130.83 114.3) (width 0.25) (layer F.Cu) (net 30) (status 30))
-  (segment (start 130.81 134.88) (end 130.81 142.24) (width 0.25) (layer F.Cu) (net 31))
+  (segment (start 139.7 143.51) (end 139.7 140.97) (width 0.25) (layer F.Cu) (net 31))
+  (segment (start 137.414 138.684) (end 130.81 138.684) (width 0.25) (layer F.Cu) (net 31))
+  (segment (start 139.7 140.97) (end 137.414 138.684) (width 0.25) (layer F.Cu) (net 31))
+  (segment (start 130.81 134.88) (end 130.81 138.684) (width 0.25) (layer F.Cu) (net 31))
+  (segment (start 130.81 138.684) (end 130.81 142.24) (width 0.25) (layer F.Cu) (net 31))
   (segment (start 130.81 142.24) (end 132.08 143.51) (width 0.25) (layer F.Cu) (net 31))
-  (segment (start 139.7 143.51) (end 139.7 142.24) (width 0.25) (layer F.Cu) (net 31) (status 30))
   (segment (start 124.46 143.51) (end 124.46 134.88) (width 0.25) (layer F.Cu) (net 32) (status 10))
   (segment (start 127 143.51) (end 127 134.88) (width 0.25) (layer F.Cu) (net 33) (status 10))
+  (segment (start 130.81 129.28) (end 130.81 125.81) (width 0.25) (layer F.Cu) (net 34))
   (segment (start 124.46 129.28) (end 124.46 125.81) (width 0.25) (layer F.Cu) (net 35) (status 20))
   (zone (net 27) (net_name 7.4V) (layer F.Cu) (hatch edge 0.508)
