File: PCBs/Recovery Board/_saved_Recovery Board.sch (KiCad schematic (older format))
At the start: 18 parts, among them J1 Conn_01x02, J2 Conn_01x02, J3 Conn_01x02, J4 Conn_01x02, J5 Conn_01x02, U1 R-78E3.3-0.5, X1 XBee-S2C

Commit message: stashing changes
Parts:
- C3: renamed from C?; value 10uF -> 1uF
- C4: renamed from C?; value 10uF -> 8.2pF
- renumbered 2k to 2k1, 3k to 3k1
Changed lines of the file:
@@
 	4600 5650 3250 5650
 $Comp
-L R 2k
+L R 2k1
 U 1 1 5A8B21DB
 P 6600 5600
-F 0 "2k" V 6680 5600 50  0000 C CNN
+F 0 "2k1" V 6680 5600 50  0000 C CNN
 F 1 "R3" V 6600 5600 50  0000 C CNN
 F 2 "Resistors_SMD:R_0805_HandSoldering" V 6530 5600 50  0001 C CNN
@@
 $EndComp
 $Comp
-L R 3k
+L R 3k1
 U 1 1 5A8B22A6
 P 6600 6300
-F 0 "3k" V 6680 6300 50  0000 C CNN
+F 0 "3k1" V 6680 6300 50  0000 C CNN
 F 1 "R4" V 6600 6300 50  0000 C CNN
 F 2 "Resistors_SMD:R_0805_HandSoldering" V 6530 6300 50  0001 C CNN
@@
 	7300 4200 7300 4300
 $Comp
-L GND #PWR?
+L GND #PWR013
 U 1 1 5ABA400A
 P 7300 4750
-F 0 "#PWR?" H 7300 4500 50  0001 C CNN
+F 0 "#PWR013" H 7300 4500 50  0001 C CNN
 F 1 "GND" H 7300 4600 50  0000 C CNN
 F 2 "" H 7300 4750 50  0001 C CNN
@@
 $EndComp
 $Comp
-L C C?
+L C C3
 U 1 1 5ABA4010
 P 7300 4450
-F 0 "C?" H 7325 4550 50  0000 L CNN
-F 1 "10uF" H 7325 4350 50  0000 L CNN
+F 0 "C3" H 7325 4550 50  0000 L CNN
+F 1 "1uF" H 7325 4350 50  0000 L CNN
 F 2 "Capacitors_SMD:C_0805_HandSoldering" H 7338 4300 50  0001 C CNN
 F 3 "" H 7300 4450 50  0001 C CNN
@@
 	7550 4200 7550 4300
 $Comp
-L GND #PWR?
+L GND #PWR014
 U 1 1 5ABA4092
 P 7550 4750
-F 0 "#PWR?" H 7550 4500 50  0001 C CNN
+F 0 "#PWR014" H 7550 4500 50  0001 C CNN
 F 1 "GND" H 7550 4600 50  0000 C CNN
 F 2 "" H 7550 4750 50  0001 C CNN
@@
 $EndComp
 $Comp
-L C C?
+L C C4
 U 1 1 5ABA4098
 P 7550 4450
-F 0 "C?" H 7575 4550 50  0000 L CNN
-F 1 "10uF" H 7575 4350 50  0000 L CNN
+F 0 "C4" H 7575 4550 50  0000 L CNN
+F 1 "8.2pF" H 7575 4350 50  0000 L CNN
 F 2 "Capacitors_SMD:C_0805_HandSoldering" H 7588 4300 50  0001 C CNN
 F 3 "" H 7550 4450 50  0001 C CNN
