File: PCBs/Recovery Board/Recovery Board.kicad_pcb (KiCad board)
At the start: 2 copper layers, 85 x 56 mm, 35 parts, among them J1 Conn_01x02, J2 Conn_01x02, J3 Conn_01x02, J4 Conn_01x02, J5 Conn_01x02, J6 Conn_01x02, J7 Conn_01x02, U1 R-78E3.3-0.5, U2 PI4ULS5V201TAEX-RESCUE-instru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, U3 PI4ULS5V201TAEX-RESCUE-instru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

Commit message: Fixed instr and recovery components per Alexs review
Added IMU current limiting resistors
Moved the caps near J4 on instr
Swapped out phototransistor footprint
Flipped I2C silk screen on J1 recovery
Flipped GND and TX silk screen on J6 recovery
renamed strat to alt on recovery silk screen
Other:
- board text added: "ALT_COMMS"
- board text added: "ALT_SW"
- board text added: "SCL SDA"
- board text added: "TX GND"
- board text removed: "ALTIMETER"
- board text removed: "GND TX"
- board text removed: "SDA SCL"
- board text removed: "STRAT"
Changed lines of the file:
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@@
     (links 62)
     (no_connects 0)
-    (area 82.924999 93.924999 168.075001 150.075001)
+    (area 77.442857 86.7212 173.557143 152.459)
     (thickness 1.6)
     (drawings 23)
@@
     (effects (font (size 1 1) (thickness 0.15)))
   )
-  (gr_text "SDA SCL" (at 148.59 147.574) (layer F.SilkS)
+  (gr_text "SCL SDA" (at 148.59 147.574) (layer F.SilkS)
     (effects (font (size 1 1) (thickness 0.15)))
   )
   (gr_circle (center 111.506 112.014) (end 111.252 112.268) (layer F.SilkS) (width 0.2))
   (gr_circle (center 113.792 134.112) (end 113.538 134.366) (layer F.SilkS) (width 0.2))
-  (gr_text "GND TX" (at 117.856 147.574) (layer F.SilkS)
+  (gr_text "TX GND" (at 117.856 147.574) (layer F.SilkS)
     (effects (font (size 1 1) (thickness 0.15)))
   )
-  (gr_text STRAT (at 118.11 139.7) (layer F.SilkS)
+  (gr_text ALT_COMMS (at 118.11 139.7) (layer F.SilkS)
     (effects (font (size 1 1) (thickness 0.15)))
   )
-  (gr_text ALTIMETER (at 125.73 139.7) (layer F.SilkS)
+  (gr_text ALT_SW (at 125.73 139.7) (layer F.SilkS)
     (effects (font (size 1 1) (thickness 0.15)))
   )
