File: PCBs/Instrumentation Board/Shifter.sch (KiCad schematic (older format))
At the start: 3 parts, among them U1 PI4ULS5V201TAEX

Commit message: Re-annotated
Parts:
- renumbered C1 to C10, C2 to C11, U1 to U8
Changed lines of the file:
@@
 $EndDescr
 $Comp
-L PI4ULS5V201TAEX U1
+L PI4ULS5V201TAEX U8
 U 1 1 5AB871B5
 P 5050 3200
-AR Path="/5AB87152/5AB871B5" Ref="U1"  Part="1"
-AR Path="/5AB8887F/5AB871B5" Ref="U1"  Part="1"
-AR Path="/5AB899BF/5AB871B5" Ref="U1"  Part="1"
-AR Path="/5AB899C9/5AB871B5" Ref="U1"  Part="1"
-AR Path="/5AB8BB45/5AB871B5" Ref="U1"  Part="1"
-AR Path="/5AB8D505/5AB871B5" Ref="U1"  Part="1"
-AR Path="/5AB8DDC4/5AB871B5" Ref="U1"  Part="1"
-F 0 "U1" H 5050 3750 60  0000 C CNN
+AR Path="/5AB87152/5AB871B5" Ref="U8"  Part="1"
+AR Path="/5AB8887F/5AB871B5" Ref="U9"  Part="1"
+AR Path="/5AB899BF/5AB871B5" Ref="U10"  Part="1"
+AR Path="/5AB899C9/5AB871B5" Ref="U11"  Part="1"
+AR Path="/5AB8BB45/5AB871B5" Ref="U12"  Part="1"
+AR Path="/5AB8D505/5AB871B5" Ref="U13"  Part="1"
+AR Path="/5AB8DDC4/5AB871B5" Ref="U14"  Part="1"
+F 0 "U14" H 5050 3750 60  0000 C CNN
 F 1 "PI4ULS5V201TAEX" H 5050 2750 60  0000 C CNN
 F 2 "" H 5050 3200 60  0001 C CNN
@@
 AR Path="/5AB8D505/5AB8720A" Ref="#PWR36"  Part="1"
 AR Path="/5AB8DDC4/5AB8720A" Ref="#PWR39"  Part="1"
-F 0 "#PWR30" H 4500 3050 50  0001 C CNN
+F 0 "#PWR39" H 4500 3050 50  0001 C CNN
 F 1 "GND" H 4500 3150 50  0000 C CNN
 F 2 "" H 4500 3300 50  0001 C CNN
@@
 AR Path="/5AB8D505/5AB87222" Ref="#PWR35"  Part="1"
 AR Path="/5AB8DDC4/5AB87222" Ref="#PWR38"  Part="1"
-F 0 "#PWR29" H 4300 3050 50  0001 C CNN
+F 0 "#PWR38" H 4300 3050 50  0001 C CNN
 F 1 "GND" H 4300 3150 50  0000 C CNN
 F 2 "" H 4300 3300 50  0001 C CNN
@@
 AR Path="/5AB8D505/5AB87230" Ref="#PWR37"  Part="1"
 AR Path="/5AB8DDC4/5AB87230" Ref="#PWR40"  Part="1"
-F 0 "#PWR31" H 5900 3300 50  0001 C CNN
+F 0 "#PWR40" H 5900 3300 50  0001 C CNN
 F 1 "GND" H 5900 3400 50  0000 C CNN
 F 2 "" H 5900 3550 50  0001 C CNN
@@
 $EndComp
 $Comp
-L C C2
+L C C11
 U 1 1 5AB8723F
 P 5900 3400
-AR Path="/5AB87152/5AB8723F" Ref="C2"  Part="1"
-AR Path="/5AB8887F/5AB8723F" Ref="C2"  Part="1"
-AR Path="/5AB899BF/5AB8723F" Ref="C2"  Part="1"
-AR Path="/5AB899C9/5AB8723F" Ref="C2"  Part="1"
-AR Path="/5AB8BB45/5AB8723F" Ref="C2"  Part="1"
-AR Path="/5AB8D505/5AB8723F" Ref="C2"  Part="1"
-AR Path="/5AB8DDC4/5AB8723F" Ref="C2"  Part="1"
-F 0 "C2" H 5925 3500 50  0000 L CNN
+AR Path="/5AB87152/5AB8723F" Ref="C11"  Part="1"
+AR Path="/5AB8887F/5AB8723F" Ref="C13"  Part="1"
+AR Path="/5AB899BF/5AB8723F" Ref="C15"  Part="1"
+AR Path="/5AB899C9/5AB8723F" Ref="C17"  Part="1"
+AR Path="/5AB8BB45/5AB8723F" Ref="C19"  Part="1"
+AR Path="/5AB8D505/5AB8723F" Ref="C21"  Part="1"
+AR Path="/5AB8DDC4/5AB8723F" Ref="C23"  Part="1"
+F 0 "C23" H 5925 3500 50  0000 L CNN
 F 1 ".1uF" H 5925 3300 50  0000 L CNN
 F 2 "" H 5938 3250 50  0001 C CNN
@@
 $EndComp
 $Comp
-L C C1
+L C C10
 U 1 1 5AB872AC
 P 4300 3150
-AR Path="/5AB87152/5AB872AC" Ref="C1"  Part="1"
-AR Path="/5AB8887F/5AB872AC" Ref="C1"  Part="1"
-AR Path="/5AB899BF/5AB872AC" Ref="C1"  Part="1"
-AR Path="/5AB899C9/5AB872AC" Ref="C1"  Part="1"
-AR Path="/5AB8BB45/5AB872AC" Ref="C1"  Part="1"
-AR Path="/5AB8D505/5AB872AC" Ref="C1"  Part="1"
-AR Path="/5AB8DDC4/5AB872AC" Ref="C1"  Part="1"
-F 0 "C1" H 4325 3250 50  0000 L CNN
+AR Path="/5AB87152/5AB872AC" Ref="C10"  Part="1"
+AR Path="/5AB8887F/5AB872AC" Ref="C12"  Part="1"
+AR Path="/5AB899BF/5AB872AC" Ref="C14"  Part="1"
+AR Path="/5AB899C9/5AB872AC" Ref="C16"  Part="1"
+AR Path="/5AB8BB45/5AB872AC" Ref="C18"  Part="1"
+AR Path="/5AB8D505/5AB872AC" Ref="C20"  Part="1"
+AR Path="/5AB8DDC4/5AB872AC" Ref="C22"  Part="1"
+F 0 "C22" H 4325 3250 50  0000 L CNN
 F 1 ".1uF" H 4325 3050 50  0000 L CNN
 F 2 "" H 4338 3000 50  0001 C CNN
