File: PCBs/Instrumentation Board/file5AB2E5F2.sch (KiCad schematic (older format))
At the start: 3 parts, among them U1 XC6201P302MR-G

Commit message: pinout changes
Connections:
- no-connect marks 3 -> 2
Other:
- moved on the sheet: C1, C2
Changed lines of the file:
@@
 LIBS:contrib
 LIBS:valves
+LIBS:a2135-h
+LIBS:ap2204k-5
+LIBS:arduino_nano
+LIBS:fgpmmopa6h
+LIBS:Recovery Board Parts
+LIBS:Recovery Board-cache
+LIBS:sot-223
 LIBS:instrumentation_board_parts
 LIBS:instrumentation_board-cache
@@
 $Descr A4 11693 8268
 encoding utf-8
-Sheet 6 10
+Sheet 2 10
 Title ""
 Date ""
@@
 L C C1
 U 1 1 5AB2EE9A
-P 3650 3350
-F 0 "C1" H 3675 3450 50  0000 L CNN
-F 1 "1uF" H 3675 3250 50  0000 L CNN
-F 2 "" H 3688 3200 50  0001 C CNN
-F 3 "" H 3650 3350 50  0001 C CNN
-	1    3650 3350
+P 4100 3350
+F 0 "C1" H 4125 3450 50  0000 L CNN
+F 1 "1uF" H 4125 3250 50  0000 L CNN
+F 2 "" H 4138 3200 50  0001 C CNN
+F 3 "" H 4100 3350 50  0001 C CNN
+	1    4100 3350
 	1    0    0    -1
 $EndComp
@@
 L GND #PWR16
 U 1 1 5AB2EEA1
-P 3650 3500
-F 0 "#PWR16" H 3650 3250 50  0001 C CNN
-F 1 "GND" H 3650 3350 50  0000 C CNN
-F 2 "" H 3650 3500 50  0001 C CNN
-F 3 "" H 3650 3500 50  0001 C CNN
-	1    3650 3500
+P 4100 3500
+F 0 "#PWR16" H 4100 3250 50  0001 C CNN
+F 1 "GND" H 4100 3350 50  0000 C CNN
+F 2 "" H 4100 3500 50  0001 C CNN
+F 3 "" H 4100 3500 50  0001 C CNN
+	1    4100 3500
 	1    0    0    -1
 $EndComp
@@
 L C C2
 U 1 1 5AB2EEA7
-P 3850 3700
-F 0 "C2" H 3875 3800 50  0000 L CNN
-F 1 "1uF" H 3875 3600 50  0000 L CNN
-F 2 "" H 3888 3550 50  0001 C CNN
-F 3 "" H 3850 3700 50  0001 C CNN
-	1    3850 3700
+P 5650 3350
+F 0 "C2" H 5675 3450 50  0000 L CNN
+F 1 "1uF" H 5675 3250 50  0000 L CNN
+F 2 "" H 5688 3200 50  0001 C CNN
+F 3 "" H 5650 3350 50  0001 C CNN
+	1    5650 3350
 	1    0    0    -1
 $EndComp
@@
 L GND #PWR17
 U 1 1 5AB2EEAE
-P 3850 3850
-F 0 "#PWR17" H 3850 3600 50  0001 C CNN
-F 1 "GND" H 3850 3700 50  0000 C CNN
-F 2 "" H 3850 3850 50  0001 C CNN
-F 3 "" H 3850 3850 50  0001 C CNN
-	1    3850 3850
+P 5650 3500
+F 0 "#PWR17" H 5650 3250 50  0001 C CNN
+F 1 "GND" H 5650 3350 50  0000 C CNN
+F 2 "" H 5650 3500 50  0001 C CNN
+F 3 "" H 5650 3500 50  0001 C CNN
+	1    5650 3500
 	1    0    0    -1
 $EndComp
@@
 L GND #PWR18
 U 1 1 5AB2EEB4
-P 5600 3300
-F 0 "#PWR18" H 5600 3050 50  0001 C CNN
-F 1 "GND" H 5600 3150 50  0000 C CNN
-F 2 "" H 5600 3300 50  0001 C CNN
-F 3 "" H 5600 3300 50  0001 C CNN
-	1    5600 3300
+P 4450 3400
+F 0 "#PWR18" H 4450 3150 50  0001 C CNN
+F 1 "GND" H 4450 3250 50  0000 C CNN
+F 2 "" H 4450 3400 50  0001 C CNN
+F 3 "" H 4450 3400 50  0001 C CNN
+	1    4450 3400
 	1    0    0    -1
 $EndComp
 NoConn ~ 5450 3350
-NoConn ~ 5450 3150
-NoConn ~ 4600 3250
 Wire Wire Line
-	4350 3700 4800 3700
+	4600 3250 4450 3250
 Wire Wire Line
-	4350 3350 4350 3700
+	4450 3250 4450 3400
+Connection ~ 4100 3150
 Wire Wire Line
-	5450 3250 5600 3250
+	4100 3150 4100 3200
 Wire Wire Line
-	5600 3250 5600 3300
-Connection ~ 4350 3550
+	3850 3150 4100 3150
 Wire Wire Line
-	3850 3550 4350 3550
-Connection ~ 3650 3150
+	4100 3150 4600 3150
+Text HLabel 3850 3150 0    60   Input ~ 0
+7.4V
+Text HLabel 5850 3150 2    60   Input ~ 0
+3V
 Wire Wire Line
-	3650 3150 3650 3200
+	5450 3150 5650 3150
 Wire Wire Line
-	3550 3150 4600 3150
+	5650 3150 5850 3150
 Wire Wire Line
-	4600 3350 4350 3350
-Text HLabel 3550 3150 0    60   Input ~ 0
-7.4V
-Text HLabel 4800 3700 2    60   Input ~ 0
-3V
+	5650 3200 5650 3150
+Connection ~ 5650 3150
+NoConn ~ 4600 3350
 $EndSCHEMATC

Commit message: Re-annotated
Parts:
- renumbered C1 to C6, C2 to C7, U1 to U6
Changed lines of the file:
@@
 $EndDescr
 $Comp
-L XC6201P302MR-G U1
+L XC6201P302MR-G U6
 U 1 1 5AB2EE92
 P 5050 3350
-F 0 "U1" H 5050 3650 60  0000 C CNN
+F 0 "U6" H 5050 3650 60  0000 C CNN
 F 1 "XC6201P302MR-G" H 5050 3250 60  0000 C CNN
 F 2 "" H 5050 3350 60  0001 C CNN
@@
 $EndComp
 $Comp
-L C C1
+L C C6
 U 1 1 5AB2EE9A
 P 4100 3350
-F 0 "C1" H 4125 3450 50  0000 L CNN
+F 0 "C6" H 4125 3450 50  0000 L CNN
 F 1 "1uF" H 4125 3250 50  0000 L CNN
 F 2 "" H 4138 3200 50  0001 C CNN
@@
 $EndComp
 $Comp
-L GND #PWR16
+L GND #PWR17
 U 1 1 5AB2EEA1
 P 4100 3500
-F 0 "#PWR16" H 4100 3250 50  0001 C CNN
+F 0 "#PWR17" H 4100 3250 50  0001 C CNN
 F 1 "GND" H 4100 3350 50  0000 C CNN
 F 2 "" H 4100 3500 50  0001 C CNN
@@
 $EndComp
 $Comp
-L C C2
+L C C7
 U 1 1 5AB2EEA7
 P 5650 3350
-F 0 "C2" H 5675 3450 50  0000 L CNN
+F 0 "C7" H 5675 3450 50  0000 L CNN
 F 1 "1uF" H 5675 3250 50  0000 L CNN
 F 2 "" H 5688 3200 50  0001 C CNN
@@
 $EndComp
 $Comp
-L GND #PWR17
+L GND #PWR18
 U 1 1 5AB2EEAE
 P 5650 3500
-F 0 "#PWR17" H 5650 3250 50  0001 C CNN
+F 0 "#PWR18" H 5650 3250 50  0001 C CNN
 F 1 "GND" H 5650 3350 50  0000 C CNN
 F 2 "" H 5650 3500 50  0001 C CNN
@@
 $EndComp
 $Comp
-L GND #PWR18
+L GND #PWR16
 U 1 1 5AB2EEB4
 P 4450 3400
-F 0 "#PWR18" H 4450 3150 50  0001 C CNN
+F 0 "#PWR16" H 4450 3150 50  0001 C CNN
 F 1 "GND" H 4450 3250 50  0000 C CNN
 F 2 "" H 4450 3400 50  0001 C CNN
@@
 	4100 3150 4100 3200
 Wire Wire Line
-	3850 3150 4100 3150
-Wire Wire Line
-	4100 3150 4600 3150
+	3850 3150 4600 3150
 Text HLabel 3850 3150 0    60   Input ~ 0
 7.4V
@@
 3V
 Wire Wire Line
-	5450 3150 5650 3150
-Wire Wire Line
-	5650 3150 5850 3150
+	5450 3150 5850 3150
 Wire Wire Line
 	5650 3200 5650 3150
