File: PCBs/Instrumentation Board/file5AB2E5F2.sch (KiCad schematic (older format))
At the start: 3 parts, among them U6 XC6201P302MR-G

Commit message: Started instrumentation Netlist
Finished footprints for shifter, regulators and IMUs
Parts:
- U6: footprint (none) -> sot:SOT-23-5
Changed lines of the file:
@@
 EESchema Schematic File Version 2
+LIBS:instrumentation_board-rescue
 LIBS:power
 LIBS:device
@@
 F 0 "U6" H 5050 3650 60  0000 C CNN
 F 1 "XC6201P302MR-G" H 5050 3250 60  0000 C CNN
-F 2 "" H 5050 3350 60  0001 C CNN
+F 2 "sot:SOT-23-5" H 5050 3350 60  0001 C CNN
 F 3 "" H 5050 3350 60  0001 C CNN
 	1    5050 3350

Commit message: review changes + instr board PCB
Parts:
- C6, C7: footprint (none) -> Capacitors_SMD:C_0805_HandSoldering
Changed lines of the file:
@@
 F 0 "C6" H 4125 3450 50  0000 L CNN
 F 1 "1uF" H 4125 3250 50  0000 L CNN
-F 2 "" H 4138 3200 50  0001 C CNN
+F 2 "Capacitors_SMD:C_0805_HandSoldering" H 4138 3200 50  0001 C CNN
 F 3 "" H 4100 3350 50  0001 C CNN
 	1    4100 3350
@@
 $EndComp
 $Comp
-L GND #PWR16
+L GND #PWR016
 U 1 1 5AB2EEA1
 P 4100 3500
-F 0 "#PWR16" H 4100 3250 50  0001 C CNN
+F 0 "#PWR016" H 4100 3250 50  0001 C CNN
 F 1 "GND" H 4100 3350 50  0000 C CNN
 F 2 "" H 4100 3500 50  0001 C CNN
@@
 F 0 "C7" H 5675 3450 50  0000 L CNN
 F 1 "1uF" H 5675 3250 50  0000 L CNN
-F 2 "" H 5688 3200 50  0001 C CNN
+F 2 "Capacitors_SMD:C_0805_HandSoldering" H 5688 3200 50  0001 C CNN
 F 3 "" H 5650 3350 50  0001 C CNN
 	1    5650 3350
@@
 $EndComp
 $Comp
-L GND #PWR18
+L GND #PWR017
 U 1 1 5AB2EEAE
 P 5650 3500
-F 0 "#PWR18" H 5650 3250 50  0001 C CNN
+F 0 "#PWR017" H 5650 3250 50  0001 C CNN
 F 1 "GND" H 5650 3350 50  0000 C CNN
 F 2 "" H 5650 3500 50  0001 C CNN
@@
 $EndComp
 $Comp
-L GND #PWR17
+L GND #PWR018
 U 1 1 5AB2EEB4
 P 4450 3400
-F 0 "#PWR17" H 4450 3150 50  0001 C CNN
+F 0 "#PWR018" H 4450 3150 50  0001 C CNN
 F 1 "GND" H 4450 3250 50  0000 C CNN
 F 2 "" H 4450 3400 50  0001 C CNN

Commit message: rerouted payload instr board and completed all changes per Alexs review
Parts:
- U6: footprint sot:SOT-23-5 -> TO_SOT_Packages_SMD:SOT-23-5_HandSoldering
Changed lines of the file:
@@
 F 0 "U6" H 5050 3650 60  0000 C CNN
 F 1 "XC6201P302MR-G" H 5050 3250 60  0000 C CNN
-F 2 "sot:SOT-23-5" H 5050 3350 60  0001 C CNN
+F 2 "TO_SOT_Packages_SMD:SOT-23-5_HandSoldering" H 5050 3350 60  0001 C CNN
 F 3 "" H 5050 3350 60  0001 C CNN
 	1    5050 3350
@@
 $EndComp
 $Comp
-L GND #PWR016
+L GND #PWR014
 U 1 1 5AB2EEA1
 P 4100 3500
-F 0 "#PWR016" H 4100 3250 50  0001 C CNN
+F 0 "#PWR014" H 4100 3250 50  0001 C CNN
 F 1 "GND" H 4100 3350 50  0000 C CNN
 F 2 "" H 4100 3500 50  0001 C CNN
@@
 $EndComp
 $Comp
-L GND #PWR017
+L GND #PWR015
 U 1 1 5AB2EEAE
 P 5650 3500
-F 0 "#PWR017" H 5650 3250 50  0001 C CNN
+F 0 "#PWR015" H 5650 3250 50  0001 C CNN
 F 1 "GND" H 5650 3350 50  0000 C CNN
 F 2 "" H 5650 3500 50  0001 C CNN
@@
 $EndComp
 $Comp
-L GND #PWR018
+L GND #PWR016
 U 1 1 5AB2EEB4
 P 4450 3400
-F 0 "#PWR018" H 4450 3150 50  0001 C CNN
+F 0 "#PWR016" H 4450 3150 50  0001 C CNN
 F 1 "GND" H 4450 3250 50  0000 C CNN
 F 2 "" H 4450 3400 50  0001 C CNN
