File: PCBs/Instrumentation Board/file5AB2F70B.sch (KiCad schematic (older format))
At the start: 3 parts, among them U1 TPS71518DCKR

Commit message: Re-annotated
Parts:
- renumbered C1 to C8, C2 to C9, U1 to U7
Changed lines of the file:
@@
 $EndDescr
 $Comp
-L TPS71518DCKR U1
+L TPS71518DCKR U7
 U 1 1 5AB2F912
 P 5150 3250
-F 0 "U1" H 5150 3550 60  0000 C CNN
+F 0 "U7" H 5150 3550 60  0000 C CNN
 F 1 "TPS71518DCKR" H 5100 3050 60  0000 C CNN
 F 2 "" H 5250 3250 60  0001 C CNN
@@
 $EndComp
 $Comp
-L C C2
+L C C9
 U 1 1 5AB2F920
 P 5850 3500
-F 0 "C2" H 5875 3600 50  0000 L CNN
+F 0 "C9" H 5875 3600 50  0000 L CNN
 F 1 ".1uF" H 5875 3400 50  0000 L CNN
 F 2 "" H 5888 3350 50  0001 C CNN
@@
 $EndComp
 $Comp
-L C C1
+L C C8
 U 1 1 5AB2F927
 P 4500 3050
-F 0 "C1" H 4525 3150 50  0000 L CNN
+F 0 "C8" H 4525 3150 50  0000 L CNN
 F 1 ".47uF" H 4525 2950 50  0000 L CNN
 F 2 "" H 4538 2900 50  0001 C CNN
