File: PCBs/Instrumentation Board/file5AB2F70B.sch (KiCad schematic (older format))
At the start: 3 parts, among them U7 TPS71518DCKR

Commit message: Started instrumentation Netlist
Finished footprints for shifter, regulators and IMUs
Parts:
- U7: footprint (none) -> sot:SOT-23-5
Changed lines of the file:
@@
 EESchema Schematic File Version 2
+LIBS:instrumentation_board-rescue
 LIBS:power
 LIBS:device
@@
 F 0 "U7" H 5150 3550 60  0000 C CNN
 F 1 "TPS71518DCKR" H 5100 3050 60  0000 C CNN
-F 2 "" H 5250 3250 60  0001 C CNN
+F 2 "sot:SOT-23-5" H 5250 3250 60  0001 C CNN
 F 3 "" H 5250 3250 60  0001 C CNN
 	1    5150 3250

Commit message: added various review changes
Parts:
- C8: value .47uF -> 0.47uF
- C9: value .1uF -> 0.1uF
Other:
- moved on the sheet: C8
Changed lines of the file:
@@
 $Descr A4 11693 8268
 encoding utf-8
-Sheet 3 10
+Sheet 3 11
 Title ""
 Date ""
@@
 $EndComp
 $Comp
-L GND #PWR019
+L GND #PWR19
 U 1 1 5AB2F91A
 P 4500 3750
-F 0 "#PWR019" H 4500 3500 50  0001 C CNN
+F 0 "#PWR19" H 4500 3500 50  0001 C CNN
 F 1 "GND" H 4500 3600 50  0000 C CNN
 F 2 "" H 4500 3750 50  0001 C CNN
@@
 P 5850 3500
 F 0 "C9" H 5875 3600 50  0000 L CNN
-F 1 ".1uF" H 5875 3400 50  0000 L CNN
+F 1 "0.1uF" H 5875 3400 50  0000 L CNN
 F 2 "" H 5888 3350 50  0001 C CNN
 F 3 "" H 5850 3500 50  0001 C CNN
@@
 L C C8
 U 1 1 5AB2F927
-P 4500 3050
-F 0 "C8" H 4525 3150 50  0000 L CNN
-F 1 ".47uF" H 4525 2950 50  0000 L CNN
-F 2 "" H 4538 2900 50  0001 C CNN
-F 3 "" H 4500 3050 50  0001 C CNN
-	1    4500 3050
+P 6500 3050
+F 0 "C8" H 6525 3150 50  0000 L CNN
+F 1 "0.47uF" H 6525 2950 50  0000 L CNN
+F 2 "" H 6538 2900 50  0001 C CNN
+F 3 "" H 6500 3050 50  0001 C CNN
+	1    6500 3050
 	1    0    0    -1
 $EndComp
@@
 	5850 2900 5850 3100
 Wire Wire Line
-	4500 2900 5850 2900
-Connection ~ 4500 3650
-Wire Wire Line
 	4500 3200 4650 3200
 Wire Wire Line
 	4500 3200 4500 3750
-Wire Wire Line
-	5850 3650 4500 3650
 Connection ~ 5850 3300
 Wire Wire Line
@@
 Text HLabel 6000 3300 2    60   Input ~ 0
 7.4V
+$Comp
+L GND #PWR20
+U 1 1 5ABF508B
+P 5850 3650
+F 0 "#PWR20" H 5850 3400 50  0001 C CNN
+F 1 "GND" H 5850 3500 50  0000 C CNN
+F 2 "" H 5850 3650 50  0001 C CNN
+F 3 "" H 5850 3650 50  0001 C CNN
+	1    5850 3650
+	1    0    0    -1
+$EndComp
+$Comp
+L GND #PWR21
+U 1 1 5ABF50F1
+P 6500 3200
+F 0 "#PWR21" H 6500 2950 50  0001 C CNN
+F 1 "GND" H 6500 3050 50  0000 C CNN
+F 2 "" H 6500 3200 50  0001 C CNN
+F 3 "" H 6500 3200 50  0001 C CNN
+	1    6500 3200
+	1    0    0    -1
+$EndComp
+Wire Wire Line
+	6500 2900 5850 2900
 $EndSCHEMATC

Commit message: swapped TX and RX pins
Parts:
- renumbered C9 to C8, C8 to C9
Changed lines of the file:
@@
 $Descr A4 11693 8268
 encoding utf-8
-Sheet 3 11
+Sheet 3 13
 Title ""
 Date ""
@@
 $EndComp
 $Comp
-L C C9
+L C C8
 U 1 1 5AB2F920
 P 5850 3500
-F 0 "C9" H 5875 3600 50  0000 L CNN
+F 0 "C8" H 5875 3600 50  0000 L CNN
 F 1 "0.1uF" H 5875 3400 50  0000 L CNN
 F 2 "" H 5888 3350 50  0001 C CNN
@@
 $EndComp
 $Comp
-L C C8
+L C C9
 U 1 1 5AB2F927
 P 6500 3050
-F 0 "C8" H 6525 3150 50  0000 L CNN
+F 0 "C9" H 6525 3150 50  0000 L CNN
 F 1 "0.47uF" H 6525 2950 50  0000 L CNN
 F 2 "" H 6538 2900 50  0001 C CNN

Commit message: review changes + instr board PCB
Parts:
- C8, C9: footprint (none) -> Capacitors_SMD:C_0805_HandSoldering
Changed lines of the file:
@@
 $EndComp
 $Comp
-L GND #PWR19
+L GND #PWR019
 U 1 1 5AB2F91A
 P 4500 3750
-F 0 "#PWR19" H 4500 3500 50  0001 C CNN
+F 0 "#PWR019" H 4500 3500 50  0001 C CNN
 F 1 "GND" H 4500 3600 50  0000 C CNN
 F 2 "" H 4500 3750 50  0001 C CNN
@@
 F 0 "C8" H 5875 3600 50  0000 L CNN
 F 1 "0.1uF" H 5875 3400 50  0000 L CNN
-F 2 "" H 5888 3350 50  0001 C CNN
+F 2 "Capacitors_SMD:C_0805_HandSoldering" H 5888 3350 50  0001 C CNN
 F 3 "" H 5850 3500 50  0001 C CNN
 	1    5850 3500
@@
 F 0 "C9" H 6525 3150 50  0000 L CNN
 F 1 "0.47uF" H 6525 2950 50  0000 L CNN
-F 2 "" H 6538 2900 50  0001 C CNN
+F 2 "Capacitors_SMD:C_0805_HandSoldering" H 6538 2900 50  0001 C CNN
 F 3 "" H 6500 3050 50  0001 C CNN
 	1    6500 3050
@@
 7.4V
 $Comp
-L GND #PWR20
+L GND #PWR020
 U 1 1 5ABF508B
 P 5850 3650
-F 0 "#PWR20" H 5850 3400 50  0001 C CNN
+F 0 "#PWR020" H 5850 3400 50  0001 C CNN
 F 1 "GND" H 5850 3500 50  0000 C CNN
 F 2 "" H 5850 3650 50  0001 C CNN
@@
 $EndComp
 $Comp
-L GND #PWR21
+L GND #PWR021
 U 1 1 5ABF50F1
 P 6500 3200
-F 0 "#PWR21" H 6500 2950 50  0001 C CNN
+F 0 "#PWR021" H 6500 2950 50  0001 C CNN
 F 1 "GND" H 6500 3050 50  0000 C CNN
 F 2 "" H 6500 3200 50  0001 C CNN

Commit message: rerouted payload instr board and completed all changes per Alexs review
Parts:
- U7: footprint sot:SOT-23-5 -> TO_SOT_Packages_SMD:SOT-23-5_HandSoldering
Changed lines of the file:
@@
 F 0 "U7" H 5150 3550 60  0000 C CNN
 F 1 "TPS71518DCKR" H 5100 3050 60  0000 C CNN
-F 2 "sot:SOT-23-5" H 5250 3250 60  0001 C CNN
+F 2 "TO_SOT_Packages_SMD:SOT-23-5_HandSoldering" H 5250 3250 60  0001 C CNN
 F 3 "" H 5250 3250 60  0001 C CNN
 	1    5150 3250
@@
 $EndComp
 $Comp
-L GND #PWR019
+L GND #PWR017
 U 1 1 5AB2F91A
 P 4500 3750
-F 0 "#PWR019" H 4500 3500 50  0001 C CNN
+F 0 "#PWR017" H 4500 3500 50  0001 C CNN
 F 1 "GND" H 4500 3600 50  0000 C CNN
 F 2 "" H 4500 3750 50  0001 C CNN
@@
 7.4V
 $Comp
-L GND #PWR020
+L GND #PWR018
 U 1 1 5ABF508B
 P 5850 3650
-F 0 "#PWR020" H 5850 3400 50  0001 C CNN
+F 0 "#PWR018" H 5850 3400 50  0001 C CNN
 F 1 "GND" H 5850 3500 50  0000 C CNN
 F 2 "" H 5850 3650 50  0001 C CNN
@@
 $EndComp
 $Comp
-L GND #PWR021
+L GND #PWR019
 U 1 1 5ABF50F1
 P 6500 3200
-F 0 "#PWR021" H 6500 2950 50  0001 C CNN
+F 0 "#PWR019" H 6500 2950 50  0001 C CNN
 F 1 "GND" H 6500 3050 50  0000 C CNN
 F 2 "" H 6500 3200 50  0001 C CNN
