File: PCBs/Instrumentation Board/instrumentation_board.sch (KiCad schematic (older format))
At the start: 17 parts, among them J1 Conn_01x02, J2 Conn_01x02, Q1 Q_Photo_NPN, U2 LSM6DS3HTR, U3 LSM6DS3HTR, U4 MicroSD-ADAFRUIT254, U5 GPS-ADAFRUIT746, U7 MS5607-02BA03

Commit message: Re-annotated
Parts:
- renumbered C4 to C1, C3 to C2, C9 to C3, C5 to C4, C8 to C5, R4 to R1, R1 to R2, R2 to R3, U2 to U1, U3 to U2, U7 to U3
Changed lines of the file:
@@
 $EndComp
 $Comp
-L GND #PWR3
+L GND #PWR5
 U 1 1 5A9B0C4F
 P 2350 2000
-F 0 "#PWR3" H 2350 1750 50  0001 C CNN
+F 0 "#PWR5" H 2350 1750 50  0001 C CNN
 F 1 "GND" H 2350 1850 50  0000 C CNN
 F 2 "" H 2350 2000 50  0001 C CNN
@@
 7.4V
 $Comp
-L GND #PWR2
+L GND #PWR15
 U 1 1 5A9B0CC8
 P 1400 6600
-F 0 "#PWR2" H 1400 6350 50  0001 C CNN
+F 0 "#PWR15" H 1400 6350 50  0001 C CNN
 F 1 "GND" H 1400 6450 50  0000 C CNN
 F 2 "" H 1400 6600 50  0001 C CNN
@@
 $EndComp
 $Comp
-L GND #PWR1
+L GND #PWR14
 U 1 1 5A9B0CDD
 P 1250 6600
-F 0 "#PWR1" H 1250 6350 50  0001 C CNN
+F 0 "#PWR14" H 1250 6350 50  0001 C CNN
 F 1 "GND" H 1250 6450 50  0000 C CNN
 F 2 "" H 1250 6600 50  0001 C CNN
@@
 $EndComp
 $Comp
-L GND #PWR5
+L GND #PWR13
 U 1 1 5A9B5B00
 P 6700 6100
-F 0 "#PWR5" H 6700 5850 50  0001 C CNN
+F 0 "#PWR13" H 6700 5850 50  0001 C CNN
 F 1 "GND" H 6700 5950 50  0000 C CNN
 F 2 "" H 6700 6100 50  0001 C CNN
@@
 $EndComp
 $Comp
-L MS5607-02BA03 U7
+L MS5607-02BA03 U3
 U 1 1 5A9E222C
 P 8400 4050
-F 0 "U7" H 8400 4450 60  0000 C CNN
+F 0 "U3" H 8400 4450 60  0000 C CNN
 F 1 "MS5607-02BA03" H 8400 3800 60  0000 C CNN
 F 2 "" H 8400 4050 60  0001 C CNN
@@
 $EndComp
 $Comp
-L C C8
+L C C5
 U 1 1 5AA0BC06
 P 7400 4200
-F 0 "C8" H 7425 4300 50  0000 L CNN
+F 0 "C5" H 7425 4300 50  0000 L CNN
 F 1 "100nF" H 7425 4100 50  0000 L CNN
 F 2 "" H 7438 4050 50  0001 C CNN
@@
 $EndComp
 $Comp
-L GND #PWR6
+L GND #PWR10
 U 1 1 5AA0BCD5
 P 7400 4350
-F 0 "#PWR6" H 7400 4100 50  0001 C CNN
+F 0 "#PWR10" H 7400 4100 50  0001 C CNN
 F 1 "GND" H 7400 4200 50  0000 C CNN
 F 2 "" H 7400 4350 50  0001 C CNN
@@
 $EndComp
 $Comp
-L GND #PWR10
+L GND #PWR11
 U 1 1 5AA0BE17
 P 7700 4350
-F 0 "#PWR10" H 7700 4100 50  0001 C CNN
+F 0 "#PWR11" H 7700 4100 50  0001 C CNN
 F 1 "GND" H 7700 4200 50  0000 C CNN
 F 2 "" H 7700 4350 50  0001 C CNN
@@
 SS
 $Comp
-L GND #PWR13
+L GND #PWR12
 U 1 1 5AA0CF85
 P 7800 5050
-F 0 "#PWR13" H 7800 4800 50  0001 C CNN
+F 0 "#PWR12" H 7800 4800 50  0001 C CNN
 F 1 "GND" H 7800 4900 50  0000 C CNN
 F 2 "" H 7800 5050 50  0001 C CNN
@@
 $EndComp
 $Comp
-L LSM6DS3HTR U2
+L LSM6DS3HTR U1
 U 1 1 5AA2036E
 P 8400 1300
-F 0 "U2" H 8400 1650 60  0000 C CNN
+F 0 "U1" H 8400 1650 60  0000 C CNN
 F 1 "LSM6DS3HTR" H 8400 850 60  0000 C CNN
 F 2 "" H 8450 1300 60  0001 C CNN
@@
 $EndComp
 $Comp
-L GND #PWR14
+L GND #PWR2
 U 1 1 5AA21112
 P 9900 1550
-F 0 "#PWR14" H 9900 1300 50  0001 C CNN
+F 0 "#PWR2" H 9900 1300 50  0001 C CNN
 F 1 "GND" H 9900 1400 50  0000 C CNN
 F 2 "" H 9900 1550 50  0001 C CNN
@@
 $EndComp
 $Comp
-L C C4
+L C C1
 U 1 1 5AA2114D
 P 9900 1400
-F 0 "C4" H 9925 1500 50  0000 L CNN
+F 0 "C1" H 9925 1500 50  0000 L CNN
 F 1 "100nF" H 9925 1300 50  0000 L CNN
 F 2 "" H 9938 1250 50  0001 C CNN
@@
 $EndComp
 $Comp
-L C C3
+L C C2
 U 1 1 5AA212DA
 P 7150 1600
-F 0 "C3" H 7175 1700 50  0000 L CNN
+F 0 "C2" H 7175 1700 50  0000 L CNN
 F 1 "100nF" H 7175 1500 50  0000 L CNN
 F 2 "" H 7188 1450 50  0001 C CNN
@@
 $EndComp
 $Comp
-L GND #PWR7
+L GND #PWR3
 U 1 1 5AA21334
 P 7150 1750
-F 0 "#PWR7" H 7150 1500 50  0001 C CNN
+F 0 "#PWR3" H 7150 1500 50  0001 C CNN
 F 1 "GND" H 7150 1600 50  0000 C CNN
 F 2 "" H 7150 1750 50  0001 C CNN
@@
 $EndComp
 $Comp
-L GND #PWR11
+L GND #PWR4
 U 1 1 5AA735F3
 P 7750 1850
-F 0 "#PWR11" H 7750 1600 50  0001 C CNN
+F 0 "#PWR4" H 7750 1600 50  0001 C CNN
 F 1 "GND" H 7750 1700 50  0000 C CNN
 F 2 "" H 7750 1850 50  0001 C CNN
@@
 INT1_1.8V
 $Comp
-L LSM6DS3HTR U3
+L LSM6DS3HTR U2
 U 1 1 5AA87733
 P 8400 2650
-F 0 "U3" H 8400 3000 60  0000 C CNN
+F 0 "U2" H 8400 3000 60  0000 C CNN
 F 1 "LSM6DS3HTR" H 8400 2200 60  0000 C CNN
 F 2 "" H 8450 2650 60  0001 C CNN
@@
 $EndComp
 $Comp
-L GND #PWR15
+L GND #PWR7
 U 1 1 5AA87752
 P 9900 2900
-F 0 "#PWR15" H 9900 2650 50  0001 C CNN
+F 0 "#PWR7" H 9900 2650 50  0001 C CNN
 F 1 "GND" H 9900 2750 50  0000 C CNN
 F 2 "" H 9900 2900 50  0001 C CNN
@@
 $EndComp
 $Comp
-L C C9
+L C C3
 U 1 1 5AA87758
 P 9900 2750
-F 0 "C9" H 9925 2850 50  0000 L CNN
+F 0 "C3" H 9925 2850 50  0000 L CNN
 F 1 "100nF" H 9925 2650 50  0000 L CNN
 F 2 "" H 9938 2600 50  0001 C CNN
@@
 $EndComp
 $Comp
-L C C5
+L C C4
 U 1 1 5AA8775E
 P 7150 2950
-F 0 "C5" H 7175 3050 50  0000 L CNN
+F 0 "C4" H 7175 3050 50  0000 L CNN
 F 1 "100nF" H 7175 2850 50  0000 L CNN
 F 2 "" H 7188 2800 50  0001 C CNN
@@
 $EndComp
 $Comp
-L GND #PWR12
+L GND #PWR9
 U 1 1 5AA8776A
 P 7750 3200
-F 0 "#PWR12" H 7750 2950 50  0001 C CNN
+F 0 "#PWR9" H 7750 2950 50  0001 C CNN
 F 1 "GND" H 7750 3050 50  0000 C CNN
 F 2 "" H 7750 3200 50  0001 C CNN
@@
 INT1_1.8V
 $Comp
-L GND #PWR9
+L GND #PWR1
 U 1 1 5AA87956
 P 7600 950
-F 0 "#PWR9" H 7600 700 50  0001 C CNN
+F 0 "#PWR1" H 7600 700 50  0001 C CNN
 F 1 "GND" H 7600 800 50  0000 C CNN
 F 2 "" H 7600 950 50  0001 C CNN
@@
 1.8V
 $Comp
-L GND #PWR4
+L GND #PWR6
 U 1 1 5AB3D6CF
 P 5050 2400
-F 0 "#PWR4" H 5050 2150 50  0001 C CNN
+F 0 "#PWR6" H 5050 2150 50  0001 C CNN
 F 1 "GND" H 5050 2250 50  0000 C CNN
 F 2 "" H 5050 2400 50  0001 C CNN
@@
 $EndComp
 $Comp
-L R R4
+L R R1
 U 1 1 5AB3D7FB
 P 5050 2250
-F 0 "R4" V 5130 2250 50  0000 C CNN
+F 0 "R1" V 5130 2250 50  0000 C CNN
 F 1 "10K" V 5050 2250 50  0000 C CNN
 F 2 "" V 4980 2250 50  0001 C CNN
@@
 INT0_5V
 $Comp
-L R R1
+L R R2
 U 1 1 5AB8F25C
 P 2950 4700
-F 0 "R1" V 3030 4700 50  0000 C CNN
+F 0 "R2" V 3030 4700 50  0000 C CNN
 F 1 "0" V 2950 4700 50  0000 C CNN
 F 2 "" V 2880 4700 50  0001 C CNN
@@
 $EndComp
 $Comp
-L R R2
+L R R3
 U 1 1 5AB8F757
 P 3250 4800
-F 0 "R2" V 3330 4800 50  0000 C CNN
+F 0 "R3" V 3330 4800 50  0000 C CNN
 F 1 "0" V 3250 4800 50  0000 C CNN
 F 2 "" V 3180 4800 50  0001 C CNN
