File: PCBs/Instrumentation Board/instrumentation_board.sch (KiCad schematic (older format))
At the start: 17 parts, among them J1 Conn_01x02, J2 Conn_01x02, Q1 Q_Photo_NPN, U1 LSM6DS3HTR, U2 LSM6DS3HTR, U3 MS5607-02BA03, U4 MicroSD-ADAFRUIT254, U5 GPS-ADAFRUIT746

Commit message: Started instrumentation Netlist
Finished footprints for shifter, regulators and IMUs
Parts:
- U1: footprint (none) -> Instrumentation Footprints:LGA-14
- U2: footprint (none) -> lga:LGA-14
Changed lines of the file:
@@
 EESchema Schematic File Version 2
+LIBS:instrumentation_board-rescue
 LIBS:power
 LIBS:device
@@
 F 0 "U1" H 8400 1650 60  0000 C CNN
 F 1 "LSM6DS3HTR" H 8400 850 60  0000 C CNN
-F 2 "" H 8450 1300 60  0001 C CNN
+F 2 "Instrumentation Footprints:LGA-14" H 8450 1300 60  0001 C CNN
 F 3 "" H 8450 1300 60  0001 C CNN
 	1    8400 1300
@@
 F 0 "U2" H 8400 3000 60  0000 C CNN
 F 1 "LSM6DS3HTR" H 8400 2200 60  0000 C CNN
-F 2 "" H 8450 2650 60  0001 C CNN
+F 2 "lga:LGA-14" H 8450 2650 60  0001 C CNN
 F 3 "" H 8450 2650 60  0001 C CNN
 	1    8400 2650

Commit message: added various review changes
Changed lines of the file:
@@
 $Descr A4 11693 8268
 encoding utf-8
-Sheet 1 10
+Sheet 1 11
 Title ""
 Date ""
@@
 $EndComp
 $Comp
-L GND #PWR01
+L GND #PWR3
 U 1 1 5A9B0C4F
 P 2350 2000
-F 0 "#PWR01" H 2350 1750 50  0001 C CNN
+F 0 "#PWR3" H 2350 1750 50  0001 C CNN
 F 1 "GND" H 2350 1850 50  0000 C CNN
 F 2 "" H 2350 2000 50  0001 C CNN
@@
 7.4V
 $Comp
-L GND #PWR02
+L GND #PWR2
 U 1 1 5A9B0CC8
 P 1400 6600
-F 0 "#PWR02" H 1400 6350 50  0001 C CNN
+F 0 "#PWR2" H 1400 6350 50  0001 C CNN
 F 1 "GND" H 1400 6450 50  0000 C CNN
 F 2 "" H 1400 6600 50  0001 C CNN
@@
 $EndComp
 $Comp
-L GND #PWR03
+L GND #PWR1
 U 1 1 5A9B0CDD
 P 1250 6600
-F 0 "#PWR03" H 1250 6350 50  0001 C CNN
+F 0 "#PWR1" H 1250 6350 50  0001 C CNN
 F 1 "GND" H 1250 6450 50  0000 C CNN
 F 2 "" H 1250 6600 50  0001 C CNN
@@
 $EndComp
 $Comp
-L GND #PWR04
+L GND #PWR5
 U 1 1 5A9B5B00
 P 6700 6100
-F 0 "#PWR04" H 6700 5850 50  0001 C CNN
+F 0 "#PWR5" H 6700 5850 50  0001 C CNN
 F 1 "GND" H 6700 5950 50  0000 C CNN
 F 2 "" H 6700 6100 50  0001 C CNN
@@
 $EndComp
 $Comp
-L GND #PWR05
+L GND #PWR8
 U 1 1 5AA0BCD5
 P 7400 4350
-F 0 "#PWR05" H 7400 4100 50  0001 C CNN
+F 0 "#PWR8" H 7400 4100 50  0001 C CNN
 F 1 "GND" H 7400 4200 50  0000 C CNN
 F 2 "" H 7400 4350 50  0001 C CNN
@@
 $EndComp
 $Comp
-L GND #PWR06
+L GND #PWR10
 U 1 1 5AA0BE17
 P 7700 4350
-F 0 "#PWR06" H 7700 4100 50  0001 C CNN
+F 0 "#PWR10" H 7700 4100 50  0001 C CNN
 F 1 "GND" H 7700 4200 50  0000 C CNN
 F 2 "" H 7700 4350 50  0001 C CNN
@@
 SS
 $Comp
-L GND #PWR07
+L GND #PWR13
 U 1 1 5AA0CF85
 P 7800 5050
-F 0 "#PWR07" H 7800 4800 50  0001 C CNN
+F 0 "#PWR13" H 7800 4800 50  0001 C CNN
 F 1 "GND" H 7800 4900 50  0000 C CNN
 F 2 "" H 7800 5050 50  0001 C CNN
@@
 $EndComp
 $Comp
-L GND #PWR08
+L GND #PWR14
 U 1 1 5AA21112
 P 9900 1550
-F 0 "#PWR08" H 9900 1300 50  0001 C CNN
+F 0 "#PWR14" H 9900 1300 50  0001 C CNN
 F 1 "GND" H 9900 1400 50  0000 C CNN
 F 2 "" H 9900 1550 50  0001 C CNN
@@
 $EndComp
 $Comp
-L GND #PWR09
+L GND #PWR6
 U 1 1 5AA21334
 P 7150 1750
-F 0 "#PWR09" H 7150 1500 50  0001 C CNN
+F 0 "#PWR6" H 7150 1500 50  0001 C CNN
 F 1 "GND" H 7150 1600 50  0000 C CNN
 F 2 "" H 7150 1750 50  0001 C CNN
@@
 $EndComp
 $Comp
-L GND #PWR010
+L GND #PWR11
 U 1 1 5AA735F3
 P 7750 1850
-F 0 "#PWR010" H 7750 1600 50  0001 C CNN
+F 0 "#PWR11" H 7750 1600 50  0001 C CNN
 F 1 "GND" H 7750 1700 50  0000 C CNN
 F 2 "" H 7750 1850 50  0001 C CNN
@@
 $EndComp
 $Comp
-L GND #PWR011
+L GND #PWR15
 U 1 1 5AA87752
 P 9900 2900
-F 0 "#PWR011" H 9900 2650 50  0001 C CNN
+F 0 "#PWR15" H 9900 2650 50  0001 C CNN
 F 1 "GND" H 9900 2750 50  0000 C CNN
 F 2 "" H 9900 2900 50  0001 C CNN
@@
 $EndComp
 $Comp
-L GND #PWR012
+L GND #PWR7
 U 1 1 5AA87764
 P 7150 3100
-F 0 "#PWR012" H 7150 2850 50  0001 C CNN
+F 0 "#PWR7" H 7150 2850 50  0001 C CNN
 F 1 "GND" H 7150 2950 50  0000 C CNN
 F 2 "" H 7150 3100 50  0001 C CNN
@@
 $EndComp
 $Comp
-L GND #PWR013
+L GND #PWR12
 U 1 1 5AA8776A
 P 7750 3200
-F 0 "#PWR013" H 7750 2950 50  0001 C CNN
+F 0 "#PWR12" H 7750 2950 50  0001 C CNN
 F 1 "GND" H 7750 3050 50  0000 C CNN
 F 2 "" H 7750 3200 50  0001 C CNN
@@
 INT1_1.8V
 $Comp
-L GND #PWR014
+L GND #PWR9
 U 1 1 5AA87956
 P 7600 950
-F 0 "#PWR014" H 7600 700 50  0001 C CNN
+F 0 "#PWR9" H 7600 700 50  0001 C CNN
 F 1 "GND" H 7600 800 50  0000 C CNN
 F 2 "" H 7600 950 50  0001 C CNN
@@
 1.8V
 $Comp
-L GND #PWR015
+L GND #PWR4
 U 1 1 5AB3D6CF
 P 5050 2400
-F 0 "#PWR015" H 5050 2150 50  0001 C CNN
+F 0 "#PWR4" H 5050 2150 50  0001 C CNN
 F 1 "GND" H 5050 2250 50  0000 C CNN
 F 2 "" H 5050 2400 50  0001 C CNN
@@
 	7000 6150 7150 6150
 NoConn ~ 7150 5750
+$Sheet
+S 3200 2350 650  300
+U 5ABF989A
+F0 "Sheet5ABF9899" 60
+F1 "file5ABF9899.sch" 60
+F2 "THERM_OUT" I R 3850 2500 60
+$EndSheet
 $EndSCHEMATC

Commit message: swapped TX and RX pins
Parts:
- A1: symbol Arduino_Nano -> Arduino_Nano-RESCUE-instrumentation_board
- renumbered C2 to C1, C4 to C2, C5 to C3, C1 to C4, C3 to C5, R2 to R1, R3 to R2, R1 to R3, U5 to U1, U1 to U2, U2 to U3, U3 to U4, U4 to U5
Connections:
- net Sheet5ABF9899/THERM_OUT: now also A1.22 (AD3/D17)
- net Sheet5ABF9899/THERM_OUT: now reaches A1.20 (AD1/D15)
- net Sheet5ABF9899/THERM_OUT: now reaches A1.21 (AD2/D16)
- no-connect marks 26 -> 23
Changed lines of the file:
@@
 $Descr A4 11693 8268
 encoding utf-8
-Sheet 1 11
+Sheet 1 13
 Title ""
 Date ""
@@
 $EndDescr
 $Comp
-L Arduino_Nano A1
+L Arduino_Nano-RESCUE-instrumentation_board A1
 U 1 1 5A9B0A95
 P 2100 5550
@@
 $EndComp
 $Comp
-L GPS U5
+L GPS U1
 U 1 1 5A9B54D4
 P 7650 6000
-F 0 "U5" H 7650 6500 60  0000 C CNN
+F 0 "U1" H 7650 6500 60  0000 C CNN
 F 1 "GPS-ADAFRUIT746" H 7650 5750 60  0000 C CNN
 F 2 "" H 7750 5900 60  0001 C CNN
@@
 $EndComp
 $Comp
-L MS5607-02BA03 U3
+L MS5607-02BA03 U4
 U 1 1 5A9E222C
 P 8400 4050
-F 0 "U3" H 8400 4450 60  0000 C CNN
+F 0 "U4" H 8400 4450 60  0000 C CNN
 F 1 "MS5607-02BA03" H 8400 3800 60  0000 C CNN
 F 2 "" H 8400 4050 60  0001 C CNN
@@
 $EndComp
 $Comp
-L C C5
+L C C3
 U 1 1 5AA0BC06
 P 7400 4200
-F 0 "C5" H 7425 4300 50  0000 L CNN
+F 0 "C3" H 7425 4300 50  0000 L CNN
 F 1 "100nF" H 7425 4100 50  0000 L CNN
 F 2 "" H 7438 4050 50  0001 C CNN
@@
 $EndComp
 $Comp
-L MicroSDBreakout U4
+L MicroSDBreakout U5
 U 1 1 5AA0C5D7
 P 8600 4950
-F 0 "U4" H 8600 5250 60  0000 C CNN
+F 0 "U5" H 8600 5250 60  0000 C CNN
 F 1 "MicroSD-ADAFRUIT254" H 8600 4650 60  0000 C CNN
 F 2 "" H 8750 4950 60  0001 C CNN
@@
 $EndComp
 $Comp
-L LSM6DS3HTR U1
+L LSM6DS3HTR U2
 U 1 1 5AA2036E
 P 8400 1300
-F 0 "U1" H 8400 1650 60  0000 C CNN
+F 0 "U2" H 8400 1650 60  0000 C CNN
 F 1 "LSM6DS3HTR" H 8400 850 60  0000 C CNN
 F 2 "Instrumentation Footprints:LGA-14" H 8450 1300 60  0001 C CNN
@@
 $EndComp
 $Comp
-L C C1
+L C C4
 U 1 1 5AA2114D
 P 9900 1400
-F 0 "C1" H 9925 1500 50  0000 L CNN
+F 0 "C4" H 9925 1500 50  0000 L CNN
 F 1 "100nF" H 9925 1300 50  0000 L CNN
 F 2 "" H 9938 1250 50  0001 C CNN
@@
 $EndComp
 $Comp
-L C C2
+L C C1
 U 1 1 5AA212DA
 P 7150 1600
-F 0 "C2" H 7175 1700 50  0000 L CNN
+F 0 "C1" H 7175 1700 50  0000 L CNN
 F 1 "100nF" H 7175 1500 50  0000 L CNN
 F 2 "" H 7188 1450 50  0001 C CNN
@@
 INT1_1.8V
 $Comp
-L LSM6DS3HTR U2
+L LSM6DS3HTR U3
 U 1 1 5AA87733
 P 8400 2650
-F 0 "U2" H 8400 3000 60  0000 C CNN
+F 0 "U3" H 8400 3000 60  0000 C CNN
 F 1 "LSM6DS3HTR" H 8400 2200 60  0000 C CNN
 F 2 "lga:LGA-14" H 8450 2650 60  0001 C CNN
@@
 $EndComp
 $Comp
-L C C3
+L C C5
 U 1 1 5AA87758
 P 9900 2750
-F 0 "C3" H 9925 2850 50  0000 L CNN
+F 0 "C5" H 9925 2850 50  0000 L CNN
 F 1 "100nF" H 9925 2650 50  0000 L CNN
 F 2 "" H 9938 2600 50  0001 C CNN
@@
 $EndComp
 $Comp
-L C C4
+L C C2
 U 1 1 5AA8775E
 P 7150 2950
-F 0 "C4" H 7175 3050 50  0000 L CNN
+F 0 "C2" H 7175 3050 50  0000 L CNN
 F 1 "100nF" H 7175 2850 50  0000 L CNN
 F 2 "" H 7188 2800 50  0001 C CNN
@@
 NoConn ~ 2800 6600
 NoConn ~ 2800 6500
-NoConn ~ 2800 6200
-NoConn ~ 2800 6100
-NoConn ~ 2800 6000
 NoConn ~ 2800 5400
 NoConn ~ 2800 5300
@@
 $EndComp
 $Comp
-L R R1
+L R R3
 U 1 1 5AB3D7FB
 P 5050 2250
-F 0 "R1" V 5130 2250 50  0000 C CNN
+F 0 "R3" V 5130 2250 50  0000 C CNN
 F 1 "10K" V 5050 2250 50  0000 C CNN
 F 2 "" V 4980 2250 50  0001 C CNN
@@
 INT0_5V
 $Comp
-L R R2
+L R R1
 U 1 1 5AB8F25C
 P 2950 4700
-F 0 "R2" V 3030 4700 50  0000 C CNN
+F 0 "R1" V 3030 4700 50  0000 C CNN
 F 1 "0" V 2950 4700 50  0000 C CNN
 F 2 "" V 2880 4700 50  0001 C CNN
@@
 $EndComp
 $Comp
-L R R3
+L R R2
 U 1 1 5AB8F757
 P 3250 4800
-F 0 "R3" V 3330 4800 50  0000 C CNN
+F 0 "R2" V 3330 4800 50  0000 C CNN
 F 1 "0" V 3250 4800 50  0000 C CNN
 F 2 "" V 3180 4800 50  0001 C CNN
@@
 NoConn ~ 7150 5750
 $Sheet
-S 3200 2350 650  300
+S 3450 5450 650  300
 U 5ABF989A
 F0 "Sheet5ABF9899" 60
 F1 "file5ABF9899.sch" 60
-F2 "THERM_OUT" I R 3850 2500 60
-$EndSheet
+F2 "THERM_OUT" I L 3450 5600 60
+$EndSheet
+$Sheet
+S 3450 5950 650  300
+U 5ABFB303
+F0 "Sheet5ABF9899" 60
+F1 "file5ABF9899.sch" 60
+F2 "THERM_OUT" I L 3450 6100 60
+$EndSheet
+$Sheet
+S 3450 6450 650  300
+U 5ABFB538
+F0 "Sheet5ABF9899" 60
+F1 "file5ABF9899.sch" 60
+F2 "THERM_OUT" I L 3450 6600 60
+$EndSheet
+Wire Wire Line
+	2800 6000 3250 6000
+Wire Wire Line
+	3250 6000 3250 5600
+Wire Wire Line
+	3250 5600 3450 5600
+Wire Wire Line
+	2800 6200 3250 6200
+Wire Wire Line
+	3250 6200 3250 6600
+Wire Wire Line
+	3250 6600 3450 6600
+Wire Wire Line
+	2800 6100 3450 6100
 $EndSCHEMATC
