File: PCBs/Instrumentation Board/instrumentation_board.kicad_pcb (KiCad board)
At the start: 2 copper layers, 65 x 104 mm, 59 parts, among them J1 Conn_01x02, J2 Conn_01x02, J3 Conn_01x02, J4 Conn_01x02, J5 Conn_01x02, Q1 TEMT6000X01, U1 GPS-ADAFRUIT746, U10 PI4ULS5V201TAEX, U11 PI4ULS5V201TAEX, U12 PI4ULS5V201TAEX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

Commit message: Current limiting resistors
Fixed structure of current limiting resistors on instr arduino
Parts:
- R11, R12: value 450 -> 470
- turned R12 to 90 degrees
Connections:
- R11 pad 1: INT0_1.8V -> Net-(R11-Pad1)
- R11 pad 2: /ICShifter5/B -> INT0_1.8V
- R12 pad 2: /ICShifter6/B -> Net-(R12-Pad2)
- U13 pad 5: /ICShifter5/B -> INT0_1.8V
- U14 pad 5: /ICShifter6/B -> INT1_1.8V
- U2 pad 4: INT0_1.8V -> Net-(R11-Pad1)
- U2 pad 9: INT1_1.8V -> Net-(R12-Pad2)
Routing:
- net INT1_1.8V: track 36.6 -> 116.6 mm, vias 3 -> 4
- net /ICShifter6/B: track 78.5 -> 0.00 mm, vias 2 -> 0
- net /ICShifter5/B: track 43.4 -> 0.00 mm, vias 2 -> 0
- net INT0_1.8V: track 34.2 -> 74.7 mm
- net Net-(R12-Pad2): track 0.00 -> 21.5 mm, vias 0 -> 2
- net Net-(R11-Pad1): track 0.00 -> 9.28 mm, vias 0 -> 2
- net GND: track 91.1 -> 97.2 mm

Commit message: Re-Exported Gerber files with .05mm solder mask clearance
Other:
- rule pad_to_mask_clearance: 25.4 -> 0.05
Changed lines of the file:
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@@
     (pad_size 3.2 3.2)
     (pad_drill 3.2)
-    (pad_to_mask_clearance 25.4)
+    (pad_to_mask_clearance 0.05)
     (aux_axis_origin 107.95 51.435)
     (visible_elements 7FFFFF7F)
