File: PCBs/Instrumentation Board/instrumentation_board.kicad_pcb (KiCad board)
At the start: 2 copper layers, 65 x 104 mm, 59 parts, among them J1 Conn_01x02, J2 Conn_01x02, J3 Conn_01x02, J4 Conn_01x02, J5 Conn_01x02, Q1 TEMT6000X01, U1 GPS-ADAFRUIT746, U10 PI4ULS5V201TAEX, U11 PI4ULS5V201TAEX, U12 PI4ULS5V201TAEX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

Commit message: New recovery gerbers
Routing:
- net /ICShifter7/VccA: track 38.5 -> 19.3 mm
- net GPS_IN: track 36.9 -> 31.3 mm
- net /ICShifter7/A: track 17.2 -> 18.0 mm
