File: PCBs/Transponder Board/shifter.sch (KiCad schematic (older format))
At the start: 3 parts

Commit message: review changes + instr board PCB
Connections:
- net VccA: now also U?.5 (EN)
- net VccB: no longer U?.5 (EN)
Changed lines of the file:
@@
 	6100 3250 6100 3650
-Wire Wire Line
-	5750 3550 6100 3550
-Connection ~ 6100 3550
 Wire Wire Line
 	4550 3450 4550 3250
@@
 Connection ~ 4550 3250
 Connection ~ 6100 3250
+Wire Wire Line
+	5750 3550 5750 4000
+Wire Wire Line
+	5750 4000 4350 4000
+Wire Wire Line
+	4350 4000 4350 3400
+Wire Wire Line
+	4350 3400 4550 3400
+Connection ~ 4550 3400
 $EndSCHEMATC

Commit message: completed layout for transponder board
Parts:
- removed U?: PI4ULS5V201TAEX, symbol PI4ULS5V201TAEX
- added U4: PI4ULS5V201TAEX, sot:SOT-23-6, symbol PI4ULS5V201TAEX-RESCUE-instrumentation_board
- C6, C7: renamed from C?; footprint (none) -> Capacitors_SMD:C_0805_HandSoldering
Connections:
- net A: now also U4.1 (A)
- net B: now also U4.5 (B)
- net GND: now also U4.2 (GND)
- net VccA: now also U4.3 (VccA), U4.6 (EN)
- net VccB: now also U4.4 (Vccb)
- no-connect marks 2 -> 0
Changed lines of the file:
@@
 LIBS:sot-223
 LIBS:instrumentation_board_parts
+LIBS:instrumentation_board-cache
 LIBS:Transponder-cache
 EELAYER 25 0
@@
 $EndDescr
 $Comp
-L PI4ULS5V201TAEX U?
-U 1 1 5AB9CBBE
-P 5300 3600
-F 0 "U?" H 5300 4150 60  0000 C CNN
-F 1 "PI4ULS5V201TAEX" H 5300 3400 60  0000 C CNN
-F 2 "" H 5300 3600 60  0001 C CNN
-F 3 "" H 5300 3600 60  0001 C CNN
-	1    5300 3600
-	1    0    0    -1
-$EndComp
-$Comp
-L C C?
+L C C7
 U 1 1 5AB9CC15
 P 6100 3800
-F 0 "C?" H 6125 3900 50  0000 L CNN
+F 0 "C7" H 6125 3900 50  0000 L CNN
 F 1 "0.1uF" H 6125 3700 50  0000 L CNN
-F 2 "" H 6138 3650 50  0001 C CNN
+F 2 "Capacitors_SMD:C_0805_HandSoldering" H 6138 3650 50  0001 C CNN
 F 3 "" H 6100 3800 50  0001 C CNN
 	1    6100 3800
@@
 $EndComp
 $Comp
-L C C?
+L C C6
 U 1 1 5AB9CC50
 P 4550 3600
-F 0 "C?" H 4575 3700 50  0000 L CNN
+F 0 "C6" H 4575 3700 50  0000 L CNN
 F 1 "0.1uF" H 4575 3500 50  0000 L CNN
-F 2 "" H 4588 3450 50  0001 C CNN
+F 2 "Capacitors_SMD:C_0805_HandSoldering" H 4588 3450 50  0001 C CNN
 F 3 "" H 4550 3600 50  0001 C CNN
 	1    4550 3600
@@
 	4500 3250 4850 3250
 $Comp
-L GND #PWR?
+L GND #PWR017
 U 1 1 5AB9CCC7
 P 6100 3950
-F 0 "#PWR?" H 6100 3700 50  0001 C CNN
+F 0 "#PWR017" H 6100 3700 50  0001 C CNN
 F 1 "GND" H 6100 3800 50  0000 C CNN
 F 2 "" H 6100 3950 50  0001 C CNN
@@
 $EndComp
 $Comp
-L GND #PWR?
+L GND #PWR018
 U 1 1 5AB9CD06
 P 4800 3750
-F 0 "#PWR?" H 4800 3500 50  0001 C CNN
+F 0 "#PWR018" H 4800 3500 50  0001 C CNN
 F 1 "GND" H 4800 3600 50  0000 C CNN
 F 2 "" H 4800 3750 50  0001 C CNN
@@
 $EndComp
 $Comp
-L GND #PWR?
+L GND #PWR019
 U 1 1 5AB9CD20
 P 4550 3750
-F 0 "#PWR?" H 4550 3500 50  0001 C CNN
+F 0 "#PWR019" H 4550 3500 50  0001 C CNN
 F 1 "GND" H 4550 3600 50  0000 C CNN
 F 2 "" H 4550 3750 50  0001 C CNN
@@
 Text HLabel 6150 3250 2    60   Input ~ 0
 VccB
-Text HLabel 5750 3450 2    60   Input ~ 0
+Text HLabel 5750 3400 2    60   Input ~ 0
 B
-Text HLabel 4850 3350 0    60   Input ~ 0
+Text HLabel 4850 3400 0    60   Input ~ 0
 A
-NoConn ~ 5750 3350
-NoConn ~ 4850 3450
 Connection ~ 4550 3250
 Connection ~ 6100 3250
@@
 	4350 3400 4550 3400
 Connection ~ 4550 3400
+$Comp
+L PI4ULS5V201TAEX-RESCUE-instrumentation_board U4
+U 1 1 5AC2E7AB
+P 5300 3600
+F 0 "U4" H 5300 4150 60  0000 C CNN
+F 1 "PI4ULS5V201TAEX" H 5300 3500 60  0000 C CNN
+F 2 "sot:SOT-23-6" H 5300 3600 60  0001 C CNN
+F 3 "" H 5300 3600 60  0001 C CNN
+	1    5300 3600
+	1    0    0    -1
+$EndComp
 $EndSCHEMATC

Commit message: transponder changes as per Alexs review
Parts:
- U4: footprint sot:SOT-23-6 -> TO_SOT_Packages_SMD:SOT-23-6_Handsoldering
Changed lines of the file:
@@
 F 0 "U4" H 5300 4150 60  0000 C CNN
 F 1 "PI4ULS5V201TAEX" H 5300 3500 60  0000 C CNN
-F 2 "sot:SOT-23-6" H 5300 3600 60  0001 C CNN
+F 2 "TO_SOT_Packages_SMD:SOT-23-6_Handsoldering" H 5300 3600 60  0001 C CNN
 F 3 "" H 5300 3600 60  0001 C CNN
 	1    5300 3600
