File: PCBs/Transponder Board/Transponder.kicad_pcb (KiCad board)
At the start: 2 copper layers, 65 x 88 mm, 28 parts, among them J1 Conn_01x02, J2 Conn_01x02, J3 Conn_01x02, J4 Conn_01x02, J5 Conn_01x02, J6 Conn_01x09, J7 Conn_01x02, U1 R-78E3.3-0.5, U2 MicroSDBreakout, U3 XBee-S2C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

Commit message: Connector Changes
Flipped the transponder jst-ph connectors
Replaced the molex footprint on recovery with the correct one
Connections:
- J2 pad 2: Net-(J1-Pad1) -> Net-(J1-Pad2)
- J7 pad 1: Net-(J1-Pad2) -> GND
- J7 pad 2: GND -> Net-(J1-Pad1)
Routing:
- net Net-(J1-Pad2): track 6.13 -> 81.8 mm, vias 0 -> 1
- net Net-(J1-Pad1): track 80.6 -> 12.0 mm, vias 1 -> 0
- net GND: track 43.8 -> 44.6 mm
Changed lines of the file:
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@@
     (links 60)
     (no_connects 0)
-    (area 52.442857 55.825 128.557143 146.275)
+    (area 57.924999 56.924999 123.075001 145.075001)
     (thickness 1.6)
     (drawings 24)
-    (tracks 295)
+    (tracks 301)
     (zones 0)
     (modules 28)
@@
       (net 26 7.4V))
     (pad 2 thru_hole circle (at 1.27 -3.048 90) (size 1.67 1.67) (drill 1.07) (layers *.Cu *.Mask)
-      (net 30 "Net-(J1-Pad1)"))
+      (net 51 "Net-(J1-Pad2)"))
   )
   (module molex:molex_kk_22-23-2021 (layer F.Cu)
@@
     )
     (pad 1 thru_hole rect (at 0 0) (size 1.2 1.7) (drill 0.75) (layers *.Cu *.Mask)
-      (net 51 "Net-(J1-Pad2)"))
+      (net 7 GND))
     (pad 2 thru_hole oval (at 2 0) (size 1.2 1.7) (drill 0.75) (layers *.Cu *.Mask)
-      (net 7 GND))
+      (net 30 "Net-(J1-Pad1)"))
     (model ${KISYS3DMOD}/Connectors_JST.3dshapes/JST_PH_B2B-PH-K_02x2.00mm_Straight.wrl
       (at (xyz 0 0 0))
@@
     (pad 1 thru_hole circle (at 0 0) (size 6.4 6.4) (drill 3.2) (layers *.Cu *.Mask))
   )
-  (gr_text "+ -" (at 82.042 59.182) (layer F.SilkS)
+  (gr_text "+ -" (at 82.042 59.182 180) (layer F.SilkS)
     (effects (font (size 1.5 1.5) (thickness 0.3)))
   )
-  (gr_text "+ -" (at 90.17 59.182) (layer F.SilkS)
+  (gr_text "+ -" (at 90.17 59.182 180) (layer F.SilkS)
     (effects (font (size 1.5 1.5) (thickness 0.3)))
   )
@@
   (segment (start 118.618 130.81) (end 118.618 126.318) (width 0.25) (layer F.Cu) (net 6))
   (segment (start 118.618 126.318) (end 118.11 125.81) (width 0.25) (layer F.Cu) (net 6))
+  (segment (start 88.9 62.738) (end 88.9 64.008) (width 0.25) (layer F.Cu) (net 7))
+  (segment (start 91.44 67.965) (end 92.075 68.6) (width 0.25) (layer F.Cu) (net 7))
+  (via (at 91.44 66.548) (size 0.6) (drill 0.4) (layers F.Cu B.Cu) (net 7))
+  (segment (start 91.44 67.965) (end 91.44 66.548) (width 0.25) (layer F.Cu) (net 7))
+  (segment (start 88.9 64.008) (end 91.44 66.548) (width 0.25) (layer F.Cu) (net 7))
   (segment (start 118.11 123.11) (end 118.11 119.38) (width 0.25) (layer F.Cu) (net 7))
   (via (at 118.11 119.38) (size 0.6) (drill 0.4) (layers F.Cu B.Cu) (net 7))
@@
   (segment (start 84.328 73.914) (end 83.566 74.676) (width 0.25) (layer F.Cu) (net 7))
   (segment (start 84.328 73.66) (end 84.328 73.914) (width 0.25) (layer F.Cu) (net 7))
-  (segment (start 90.9 62.738) (end 91.44 63.278) (width 0.25) (layer F.Cu) (net 7))
-  (segment (start 91.44 67.965) (end 91.44 66.548) (width 0.25) (layer F.Cu) (net 7))
-  (via (at 91.44 66.548) (size 0.6) (drill 0.4) (layers F.Cu B.Cu) (net 7))
-  (segment (start 91.44 67.965) (end 92.075 68.6) (width 0.25) (layer F.Cu) (net 7))
-  (segment (start 91.44 63.278) (end 91.44 66.548) (width 0.25) (layer F.Cu) (net 7))
   (segment (start 81.915 68.6) (end 83.546 68.6) (width 0.25) (layer F.Cu) (net 7))
   (via (at 85.598 66.548) (size 0.6) (drill 0.4) (layers F.Cu B.Cu) (net 7))
@@
   (segment (start 89.535 83.82) (end 89.535 86.995) (width 0.25) (layer F.Cu) (net 29))
   (segment (start 89.535 86.995) (end 89.535 88.92) (width 0.25) (layer F.Cu) (net 29))
-  (segment (start 80.772 62.738) (end 73.152 62.738) (width 0.25) (layer F.Cu) (net 30))
-  (via (at 71.755 71.12) (size 0.6) (drill 0.4) (layers F.Cu B.Cu) (net 30))
-  (segment (start 69.85 73.025) (end 71.755 71.12) (width 0.25) (layer B.Cu) (net 30))
-  (segment (start 69.85 128.27) (end 69.85 73.025) (width 0.25) (layer B.Cu) (net 30))
-  (segment (start 68.58 129.54) (end 69.85 128.27) (width 0.25) (layer B.Cu) (net 30))
-  (segment (start 68.58 129.54) (end 64.262 129.54) (width 0.25) (layer B.Cu) (net 30))
-  (segment (start 71.755 64.135) (end 73.152 62.738) (width 0.25) (layer F.Cu) (net 30))
-  (segment (start 71.755 71.12) (end 71.755 64.135) (width 0.25) (layer F.Cu) (net 30))
+  (segment (start 80.772 62.738) (end 80.772 62.103) (width 0.25) (layer F.Cu) (net 30))
+  (segment (start 80.772 62.103) (end 81.915 60.96) (width 0.25) (layer F.Cu) (net 30))
+  (segment (start 89.122 60.96) (end 90.9 62.738) (width 0.25) (layer F.Cu) (net 30))
+  (segment (start 81.915 60.96) (end 89.122 60.96) (width 0.25) (layer F.Cu) (net 30))
   (segment (start 92.71 100.965) (end 89.535 100.965) (width 0.25) (layer F.Cu) (net 31))
   (segment (start 91.6178 108.46054) (end 94.10446 108.46054) (width 0.25) (layer F.Cu) (net 31) (status 20))
@@
   (via (at 90.17 73.66) (size 0.6) (drill 0.4) (layers F.Cu B.Cu) (net 34))
   (segment (start 90.17 73.66) (end 88.095 73.66) (width 0.25) (layer F.Cu) (net 34))
-  (segment (start 82.772 62.738) (end 88.9 62.738) (width 0.25) (layer F.Cu) (net 51))
+  (segment (start 71.755 66.675) (end 71.755 66.04) (width 0.25) (layer F.Cu) (net 51))
+  (segment (start 81.28 64.77) (end 82.772 63.278) (width 0.25) (layer F.Cu) (net 51))
+  (segment (start 73.025 64.77) (end 81.28 64.77) (width 0.25) (layer F.Cu) (net 51))
+  (segment (start 71.755 66.04) (end 73.025 64.77) (width 0.25) (layer F.Cu) (net 51))
+  (segment (start 82.772 63.278) (end 82.772 62.738) (width 0.25) (layer F.Cu) (net 51))
+  (via (at 71.755 71.12) (size 0.6) (drill 0.4) (layers F.Cu B.Cu) (net 51))
+  (segment (start 69.85 73.025) (end 71.755 71.12) (width 0.25) (layer B.Cu) (net 51))
+  (segment (start 71.755 71.12) (end 71.755 66.675) (width 0.25) (layer F.Cu) (net 51))
+  (segment (start 69.85 128.27) (end 69.85 73.025) (width 0.25) (layer B.Cu) (net 51))
+  (segment (start 68.58 129.54) (end 69.85 128.27) (width 0.25) (layer B.Cu) (net 51))
+  (segment (start 68.58 129.54) (end 64.262 129.54) (width 0.25) (layer B.Cu) (net 51))
   (zone (net 7) (net_name GND) (layer B.Cu) (hatch edge 0.508)
     (connect_pads (clearance 0.508))

Commit message: Added zips for gerber files
Other:
- rule pad_to_mask_clearance: 0.0508 -> 0.05
Changed lines of the file:
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@@
     (links 60)
     (no_connects 0)
-    (area 57.924999 56.924999 123.075001 145.075001)
+    (area 52.442857 55.825 128.557143 146.275)
     (thickness 1.6)
     (drawings 24)
@@
     (pad_size 1.524 1.524)
     (pad_drill 0.762)
-    (pad_to_mask_clearance 0.0508)
+    (pad_to_mask_clearance 0.05)
     (aux_axis_origin 0 0)
     (visible_elements 7FFFFF7F)
